File: Hardware/JMP_SYSTEM/PowerManagaement.kicad_sch (KiCad schematic)
At the start: 0 parts

Commit message: Schematics and PCB layout
Parts:
- added BT1: 4.2V, Connector_PinHeader_2.54mm:PinHeader_1x02_P2.54mm_Vertical, symbol Device:Battery_Cell
- added C11, C12, C13: 1uF, Capacitor_SMD:C_0805_2012Metric, symbol Device:C_Small
- added J10, J11: Debug, Connector_PinHeader_2.54mm:PinHeader_1x02_P2.54mm_Vertical, symbol Connector_Generic:Conn_01x02
- added R21, R22: R em M, Resistor_SMD:R_0805_2012Metric_Pad1.20x1.40mm_HandSolder, symbol Device:R_Small
- added U3: TP4056_MODULE, adelson:Módulo_TP4056, symbol adelson:TP4056_MODULE
- added U4: Modulo_DC-DC_Boost_XL6009, adelson:Modulo_DC-DC_Boost_XL6009, symbol adelson:Modulo_DC-DC_Boost_XL6009
Connections:
- new net: J10.1 (Pin_1), U3.3 (OUT+)
- new net: C11.1, J10.2 (Pin_2), U4.1 (IN+)
- new net: C12.1, U3.5 (OUT-), U4.2 (IN-)
- new net: J11.1 (Pin_1), U4.3 (OUT+)
- new net 5V: C13.1, J11.2 (Pin_2)
- new net B+: BT1.1 (+), R21.1, U3.4 (B+)
- new net B+_AD_IN: R21.2, R22.2
- new net B-_AD_IN: BT1.2 (-), R22.1, U3.6 (B-)
- new net GNDA: C11.2, C12.2, C13.2, U4.4 (OUT-)
- no-connect marks 0 -> 2
Other:
- note added: "Alimentação por USB @ 5V"
- note added: "Modulo rele arduino Length 43 mm Width 17.5 mm Height 17 mm"
- note added: "TP4056 DIMENSIONS: 25x19x5mm (LxWxT) XL6009 BOOST: 43,18x21,082mm"
- note added: "XL6009 BOOST: https://www.sunrom.com/p/step-up-dc-dc-based-on-xl6009"
- note removed: "TP4056 + um stepUP de 3v3 - 5V"
