File: Hardware/JMP_SYSTEM/PowerManagaement.kicad_sch (KiCad schematic)
At the start: 11 parts, among them J10 Debug, J11 Debug, U3 TP4056_MODULE, U4 Modulo_DC-DC_Boost_XL6009

Commit message: Roteamento considerando I2C e Display em conjunto. O display ficara suspenso. Adicionado molex em todos os conectores. Debugs sao pinos convencionais
Parts:
- removed C12: R0, Capacitor_SMD:C_0805_2012Metric, symbol Device:C_Small
- Bateria1: renamed from BT1; footprint Connector_PinHeader_2.54mm:PinHeader_1x02_P2.54mm_Vertical -> Connector_Molex:Molex_KK-254_AE-6410-02A_1x02_P2.54mm_Vertical
Connections:
- net GNDA: now also U3.5 (OUT-), U4.2 (IN-)
Changed lines of the file:
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@@
+    (stroke (width 0) (type default) (color 0 0 0 0))
+  )
+  (wire (pts (xy 85.09 46.99) (xy 100.33 46.99))
     (stroke (width 0) (type default) (color 0 0 0 0))
   )
@@
     (stroke (width 0) (type default) (color 0 0 0 0))
   )
+  (wire (pts (xy 85.09 46.99) (xy 85.09 53.34))
+    (stroke (width 0) (type default) (color 0 0 0 0))
+  )
   (wire (pts (xy 91.44 73.66) (xy 96.52 73.66))
     (stroke (width 0) (type default) (color 0 0 0 0))
@@
     (stroke (width 0) (type default) (color 0 0 0 0))
   )
-  (wire (pts (xy 85.09 52.07) (xy 85.09 53.34))
-    (stroke (width 0) (type default) (color 0 0 0 0))
-  )
-  (wire (pts (xy 85.09 46.99) (xy 100.33 46.99))
+  (wire (pts (xy 71.12 46.99) (xy 85.09 46.99))
     (stroke (width 0) (type default) (color 0 0 0 0))
   )
@@
   )
   (polyline (pts (xy 44.45 41.91) (xy 44.45 44.45))
-    (stroke (width 0) (type default) (color 0 0 0 0))
-  )
-  (wire (pts (xy 71.12 46.99) (xy 85.09 46.99))
     (stroke (width 0) (type default) (color 0 0 0 0))
   )
@@
   (symbol (lib_id "Device:Battery_Cell") (at 78.74 80.01 0) (unit 1)
     (in_bom yes) (on_board yes)
-    (property "Reference" "BT1" (id 0) (at 72.517 75.311 0))
+    (property "Reference" "Bateria1" (id 0) (at 72.517 75.311 0))
     (property "Value" "4.2V" (id 1) (at 73.279 77.851 0))
-    (property "Footprint" "Connector_PinHeader_2.54mm:PinHeader_1x02_P2.54mm_Vertical" (id 2) (at 78.74 78.486 90)
+    (property "Footprint" "Connector_Molex:Molex_KK-254_AE-6410-02A_1x02_P2.54mm_Vertical" (id 2) (at 78.74 78.486 90)
       (effects (font (size 1.27 1.27)) hide)
     )
@@
       (effects (font (size 1.27 1.27)) hide)
     )
-    (pin "1")
-    (pin "2")
-  )
-  (symbol (lib_id "Device:C_Small") (at 85.09 49.53 0) (unit 1)
-    (in_bom yes) (on_board yes) (fields_autoplaced)
-    (property "Reference" "C12" (id 0) (at 87.63 48.2662 0)
-      (effects (font (size 1.27 1.27)) (justify left))
-    )
-    (property "Value" "R0" (id 1) (at 87.63 50.8062 0)
-      (effects (font (size 1.27 1.27)) (justify left))
-    )
-    (property "Footprint" "Capacitor_SMD:C_0805_2012Metric" (id 2) (at 85.09 49.53 0)
-      (effects (font (size 1.27 1.27)) hide)
-    )
-    (property "Datasheet" "~" (id 3) (at 85.09 49.53 0)
-      (effects (font (size 1.27 1.27)) hide)
-    )
