File: Hardware/JMP_SYSTEM/JMP_SYSTEM.kicad_sch (KiCad schematic)
At the start: 15 parts

Commit message: Schematics and PCB layout
Parts:
- removed J?: 4V, symbol Connector_Generic:Conn_01x01
- removed J?: GNDA, symbol Connector_Generic:Conn_01x01
- removed J?: 3V3, symbol Connector_Generic:Conn_01x01
- removed J?: 5V, symbol Connector_Generic:Conn_01x01
- removed RV?: R_Potentiometer, symbol Device:R_Potentiometer
- added J13, J8: Port_access, Connector_PinHeader_2.54mm:PinHeader_1x05_P2.54mm_Vertical, symbol Connector_Generic:Conn_01x05
- added J14, J19, J21: Port_access, Connector_PinHeader_2.54mm:PinHeader_1x04_P2.54mm_Vertical, symbol Connector_Generic:Conn_01x04
- added J15, J16, J17, J18, J20: Port_access, Connector_PinHeader_2.54mm:PinHeader_1x02_P2.54mm_Vertical, symbol Connector_Generic:Conn_01x02
- added J2, J3, J6, J7: Debug, Connector_PinHeader_2.54mm:PinHeader_1x02_P2.54mm_Vertical, symbol Connector_Generic:Conn_01x02
- J4: renamed from J?; footprint (none) -> Connector_PinHeader_2.54mm:PinHeader_1x04_P2.54mm_Vertical
- J5: renamed from J?; footprint (none) -> Connector_PinHeader_2.54mm:PinHeader_1x06_P2.54mm_Vertical
- gave numbers to parts that had none: 8
Connections:
- net GNDD is gone; now on net GNDA: C1.2, C2.2, J4.4 (Pin_4), J5.6 (Pin_6), SW1.1, SW2.1
- net CS: now also J19.1 (Pin_1)
- net MISO: now also J19.3 (Pin_3)
- net MOSI: now also J19.4 (Pin_4)
- net RELE: now also J14.2 (Pin_2)
- net SCK: now also J19.2 (Pin_2)
- net SENSOR_1: now also J17.1 (Pin_1), J17.2 (Pin_2)
- net SENSOR_2: now also J18.1 (Pin_1), J18.2 (Pin_2)
- removed net +5V: J4.3 (Pin_3), J5.5 (Pin_5), R1.1, R3.1
- new net: J6.1 (Pin_1), R1.1
- new net: J2.2 (Pin_2), J5.5 (Pin_5)
- new net: J3.2 (Pin_2), J4.3 (Pin_3)
- new net: J7.1 (Pin_1), R3.1
- new net 3V3: J6.2 (Pin_2), J7.2 (Pin_2)
- new net 5V: J2.1 (Pin_1), J3.1 (Pin_1)
- new net B+_AD_IN: J16.1 (Pin_1)
- new net B-_AD_IN: J16.2 (Pin_2)
- new net BT_DOWN: J21.1 (Pin_1)
- new net BT_LEFT: J21.2 (Pin_2)
- new net BT_MENU: J8.4 (Pin_4)
- new net BT_OK: J8.3 (Pin_3)
- new net BT_RIGHT: J21.4 (Pin_4)
- new net BT_RST: J13.1 (Pin_1)
- new net BT_STOP: J8.2 (Pin_2)
- new net BT_UP: J21.3 (Pin_3)
- new net PA4: J15.1 (Pin_1)
- new net PA5: J15.2 (Pin_2)
- new net PA8: J8.5 (Pin_5)
- new net PB0: J13.5 (Pin_5)
- new net PB1: J13.4 (Pin_4)
- new net PB10: J13.3 (Pin_3)
- new net PB11: J13.2 (Pin_2)
- new net PB4: J8.1 (Pin_1)
- new net PC13: J14.3 (Pin_3)
- new net PC15: J14.1 (Pin_1)
- new net SCL: J20.2 (Pin_2)
- new net SDA: J20.1 (Pin_1)
- new net VBAT: J14.4 (Pin_4)
Other:
- sheet PowerManagaement ports: added B+_AD_IN, B-_AD_IN; removed none
- sheet User _IO ports: added BT_DOWN, BT_LEFT, BT_OK, BT_RIGHT, BT_RST, BT_UP, RELE, SCL, SDA; removed A, BT_AVANCAR, BT_INSERT, BT_SELECT, DB0, DB1, DB2, DB3, DB4, DB5, DB6, DB7, E, K, RS, R/~{W}, V0
- note added: "ALIMENTAÇÃO"
- note added: "I/O DEBUG"
- note removed: "ALIMETAÇÃO (PENDENTE)"
- moved on the sheet: J4, J5, R1, R2, R4, SW1

Commit message: Roteamento considerando I2C e Display em conjunto. O display ficara suspenso. Adicionado molex em todos os conectores. Debugs sao pinos convencionais
Parts:
- removed J14, J19: Port_access, Connector_PinHeader_2.54mm:PinHeader_1x04_P2.54mm_Vertical, symbol Connector_Generic:Conn_01x04
- removed J15: Port_access, Connector_PinHeader_2.54mm:PinHeader_1x02_P2.54mm_Vertical, symbol Connector_Generic:Conn_01x02
- removed J8: Port_access, Connector_PinHeader_2.54mm:PinHeader_1x05_P2.54mm_Vertical, symbol Connector_Generic:Conn_01x05
- added J14: Ports, Connector_Molex:Molex_KK-254_AE-6410-03A_1x03_P2.54mm_Vertical, symbol Connector_Generic:Conn_01x03
- added J19: Ports, Connector_Molex:Molex_KK-254_AE-6410-05A_1x05_P2.54mm_Vertical, symbol Connector_Generic:Conn_01x05
- added J23, J9: Debug, Connector_PinHeader_2.54mm:PinHeader_1x02_P2.54mm_Vertical, symbol Connector_Generic:Conn_01x02
- added J8: Ports, Connector_Molex:Molex_KK-254_AE-6410-04A_1x04_P2.54mm_Vertical, symbol Connector_Generic:Conn_01x04
- J13: value Port_access -> Ports; footprint Connector_PinHeader_2.54mm:PinHeader_1x05_P2.54mm_Vertical -> Connector_Molex:Molex_KK-254_AE-6410-05A_1x05_P2.54mm_Vertical
- J16, J17, J18, J20: value Port_access -> Ports; footprint Connector_PinHeader_2.54mm:PinHeader_1x02_P2.54mm_Vertical -> Connector_Molex:Molex_KK-254_AE-6410-02A_1x02_P2.54mm_Vertical
- J21: value Port_access -> Ports; footprint Connector_PinHeader_2.54mm:PinHeader_1x04_P2.54mm_Vertical -> Connector_Molex:Molex_KK-254_AE-6410-04A_1x04_P2.54mm_Vertical
- J4: footprint Connector_PinHeader_2.54mm:PinHeader_1x04_P2.54mm_Vertical -> Connector_Molex:Molex_KK-254_AE-6410-04A_1x04_P2.54mm_Vertical
- J5: footprint Connector_PinHeader_2.54mm:PinHeader_1x06_P2.54mm_Vertical -> Connector_Molex:Molex_KK-254_AE-6410-06A_1x06_P2.54mm_Vertical
Connections:
- net B+_AD_IN: now also J16.2 (Pin_2); no longer J16.1 (Pin_1)
- net B-_AD_IN: now also J16.1 (Pin_1); no longer J16.2 (Pin_2)
- net BT_MENU: now also J8.4 (Pin_4)
- net BT_OK: now also J8.3 (Pin_3)
- net BT_RST: now also J13.5 (Pin_5); no longer J13.1 (Pin_1)
- net BT_STOP: now also J8.2 (Pin_2)
- net CS: now also J19.5 (Pin_5)
- net GNDA: now also J4.1 (Pin_1), J23.1 (Pin_1), J9.1 (Pin_1); no longer J4.4 (Pin_4)
- net MISO: now also J19.3 (Pin_3)
- net MOSI: now also J19.4 (Pin_4)
- net PB0: now also J13.1 (Pin_1); no longer J13.5 (Pin_5)
- net PB1: now also J13.2 (Pin_2); no longer J13.4 (Pin_4)
- net PB11: now also J13.4 (Pin_4); no longer J13.2 (Pin_2)
- net PB4: now also J8.1 (Pin_1)
- net PC13: now also J14.2 (Pin_2)
- net RELE: now also J14.3 (Pin_3)
- net RX: now also J4.4 (Pin_4); no longer J4.1 (Pin_1)
- net SCK: now also J19.2 (Pin_2)
- net TX: now also J4.3 (Pin_3); no longer J4.2 (Pin_2)
- net VBAT: now also J14.1 (Pin_1)
- net at R1.2, R2.1, SW1.2: now also J9.2 (Pin_2)
- net at J3.2 (Pin_2): now also J4.2 (Pin_2); no longer J4.3 (Pin_3)
- net at R3.2, R4.1, SW2.2: now also J23.2 (Pin_2)
- new net PB12: J19.1 (Pin_1)
Other:
- sheet BLUEPILL_STM32 ports: added LED_1, LED_2, LED_3; removed PA4, PA5, PC15
- sheet User _IO ports: added LED_1, LED_2, LED_3; removed none
- moved on the sheet: J13, J16, J17, J18, J20, J21
