File: Hardware/Core_HW/Core_HW.kicad_pcb (KiCad board)
At the start: 2 copper layers, 87.6 x 98.4 mm, 63 parts, among them J1 Debug, J10 Port_access, J11 Port_access, J12 Port_access, J13 Port_access, J14 RELE, J15 Port_access, J16 Port_access, J17 Port_access, J18 Port_access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

Commit message: geracao de gebers
Parts:
- J10, J11, J12, J13, J15, J16, J17, J18, J19, J23, J9: value Port_access -> Ports
Connections:
- net GNDD renamed GNDA
