File: Hardware/Core_HW/Core_HW.kicad_sch (KiCad schematic)
At the start: 63 parts, among them J1 Debug, J10 Port_access, J11 Port_access, J12 Port_access, J13 Port_access, J14 RELE, J15 Port_access, J16 Port_access, J17 Port_access, J18 Port_access, J19 Port_access, J2 Debug, J21 JUMP, J22 JUMP, J23 Port_access, J24 Debug, J3 BLUETOOTH, J4 MODULO SD, J5 Interface, J6 BLACKPILL, J7 Debug, J8 Debug, J9 Port_access, SW1 BT_LEFT, SW10 BT_RST, SW2 BT_RIGHT, SW3 BT_UP, SW4 BT_DOWN, SW5 BT_STOP, SW6 SENSOR, SW7 BT_MENU, SW8 SENSOR, SW9 BT_OK

Commit message: geracao de gebers
Parts:
- J10, J11, J12, J13, J15, J16, J17, J18, J19, J23, J9: value Port_access -> Ports
Changed lines of the file:
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@@
       (effects (font (size 1.27 1.27)) (justify left))
     )
-    (property "Value" "Port_access" (id 1) (at 218.313 106.426 0)
+    (property "Value" "Ports" (id 1) (at 218.313 106.426 0)
       (effects (font (size 1.27 1.27)) (justify left))
     )
@@
       (effects (font (size 1.27 1.27)) (justify left))
     )
-    (property "Value" "Port_access" (id 1) (at 241.046 111.633 0)
+    (property "Value" "Ports" (id 1) (at 247.015 104.775 0)
       (effects (font (size 1.27 1.27)) (justify left))
     )
@@
   (symbol (lib_id "Connector_Generic:Conn_01x02") (at 266.7 123.825 0) (unit 1)
     (in_bom yes) (on_board yes) (fields_autoplaced)
-    (property "Reference" "J18" (id 0) (at 269.367 123.8249 0)
-      (effects (font (size 1.27 1.27)) (justify left))
-    )
-    (property "Value" "Port_access" (id 1) (at 269.367 126.3649 0)
+    (property "Reference" "J18" (id 0) (at 269.24 123.8249 0)
+      (effects (font (size 1.27 1.27)) (justify left))
+    )
+    (property "Value" "Ports" (id 1) (at 269.24 126.3649 0)
       (effects (font (size 1.27 1.27)) (justify left))
     )
@@
       (effects (font (size 1.27 1.27)) (justify left))
     )
-    (property "Value" "Port_access" (id 1) (at 220.218 135.001 0)
+    (property "Value" "Ports" (id 1) (at 220.218 135.001 0)
       (effects (font (size 1.27 1.27)) (justify left))
     )
@@
   (symbol (lib_id "Connector_Generic:Conn_01x02") (at 266.7 130.81 0) (unit 1)
     (in_bom yes) (on_board yes) (fields_autoplaced)
-    (property "Reference" "J19" (id 0) (at 269.494 130.8099 0)
-      (effects (font (size 1.27 1.27)) (justify left))
-    )
-    (property "Value" "Port_access" (id 1) (at 269.494 133.3499 0)
+    (property "Reference" "J19" (id 0) (at 269.24 130.8099 0)
+      (effects (font (size 1.27 1.27)) (justify left))
+    )
+    (property "Value" "Ports" (id 1) (at 269.24 133.3499 0)
       (effects (font (size 1.27 1.27)) (justify left))
     )
@@
       (effects (font (size 1.27 1.27)) (justify left))
     )
-    (property "Value" "Port_access" (id 1) (at 237.49 121.285 0)
+    (property "Value" "Ports" (id 1) (at 237.49 121.285 0)
       (effects (font (size 1.27 1.27)) (justify left))
     )
@@
       (effects (font (size 1.27 1.27)) (justify left))
     )
-    (property "Value" "Port_access" (id 1) (at 219.456 120.015 0)
+    (property "Value" "Ports" (id 1) (at 219.456 120.015 0)
       (effects (font (size 1.27 1.27)) (justify left))
     )
@@
       (effects (font (size 1.27 1.27)) (justify left))
     )
-    (property "Value" "Port_access" (id 1) (at 241.3 133.985 0)
+    (property "Value" "Ports" (id 1) (at 241.3 133.985 0)
       (effects (font (size 1.27 1.27)) (justify left))
     )
@@
   (symbol (lib_id "Connector_Generic:Conn_01x02") (at 266.065 107.95 0) (unit 1)
     (in_bom yes) (on_board yes) (fields_autoplaced)
-    (property "Reference" "J16" (id 0) (at 268.732 107.9499 0)
-      (effects (font (size 1.27 1.27)) (justify left))
-    )
-    (property "Value" "Port_access" (id 1) (at 268.732 110.4899 0)
+    (property "Reference" "J16" (id 0) (at 269.24 107.9499 0)
+      (effects (font (size 1.27 1.27)) (justify left))
+    )
+    (property "Value" "Ports" (id 1) (at 269.24 110.4899 0)
       (effects (font (size 1.27 1.27)) (justify left))
     )
@@
   (symbol (lib_id "Connector_Generic:Conn_01x02") (at 266.7 116.84 0) (unit 1)
     (in_bom yes) (on_board yes) (fields_autoplaced)
-    (property "Reference" "J17" (id 0) (at 269.367 116.8399 0)
-      (effects (font (size 1.27 1.27)) (justify left))
-    )
-    (property "Value" "Port_access" (id 1) (at 269.367 119.3799 0)
+    (property "Reference" "J17" (id 0) (at 269.24 116.8399 0)
+      (effects (font (size 1.27 1.27)) (justify left))
+    )
+    (property "Value" "Ports" (id 1) (at 269.24 119.3799 0)
       (effects (font (size 1.27 1.27)) (justify left))
     )
@@
   (symbol (lib_id "Connector_Generic:Conn_01x02") (at 266.065 99.695 0) (unit 1)
     (in_bom yes) (on_board yes) (fields_autoplaced)
-    (property "Reference" "J15" (id 0) (at 268.732 99.6949 0)
-      (effects (font (size 1.27 1.27)) (justify left))
-    )
-    (property "Value" "Port_access" (id 1) (at 268.732 102.2349 0)
+    (property "Reference" "J15" (id 0) (at 269.24 99.6949 0)
+      (effects (font (size 1.27 1.27)) (justify left))
+    )
+    (property "Value" "Ports" (id 1) (at 269.24 102.2349 0)
       (effects (font (size 1.27 1.27)) (justify left))
     )
@@
     )
     (path "/0a546429-7348-41ea-adbf-e47774926f37"
-      (reference "J9") (unit 1) (value "Port_access") (footprint "Connector_PinHeader_2.54mm:PinHeader_1x04_P2.54mm_Vertical")
+      (reference "J9") (unit 1) (value "Ports") (footprint "Connector_PinHeader_2.54mm:PinHeader_1x04_P2.54mm_Vertical")
     )
     (path "/c5b389d1-233d-4908-a78c-6f69f79dce70"
-      (reference "J10") (unit 1) (value "Port_access") (footprint "Connector_PinHeader_2.54mm:PinHeader_1x04_P2.54mm_Vertical")
+      (reference "J10") (unit 1) (value "Ports") (footprint "Connector_PinHeader_2.54mm:PinHeader_1x04_P2.54mm_Vertical")
     )
     (path "/6a745364-661e-4dff-8758-bcacd2fb1249"
-      (reference "J11") (unit 1) (value "Port_access") (footprint "Connector_PinHeader_2.54mm:PinHeader_1x04_P2.54mm_Vertical")
+      (reference "J11") (unit 1) (value "Ports") (footprint "Connector_PinHeader_2.54mm:PinHeader_1x04_P2.54mm_Vertical")
     )
     (path "/a9263f09-7b7e-41ae-8554-bb66bd7c2b2a"
-      (reference "J12") (unit 1) (value "Port_access") (footprint "Connector_PinHeader_2.54mm:PinHeader_1x02_P2.54mm_Vertical")
+      (reference "J12") (unit 1) (value "Ports") (footprint "Connector_PinHeader_2.54mm:PinHeader_1x02_P2.54mm_Vertical")
     )
     (path "/237a0ae8-e1d9-4f9b-9d08-328331f793bb"
-      (reference "J13") (unit 1) (value "Port_access") (footprint "Connector_PinHeader_2.54mm:PinHeader_1x05_P2.54mm_Vertical")
+      (reference "J13") (unit 1) (value "Ports") (footprint "Connector_PinHeader_2.54mm:PinHeader_1x05_P2.54mm_Vertical")
     )
     (path "/72494d27-94de-4c78-9684-fbdfee3e0376"
@@
     )
     (path "/fbef6213-ee81-4d61-a0d9-e5633486d967"
-      (reference "J15") (unit 1) (value "Port_access") (footprint "Connector_PinHeader_2.54mm:PinHeader_1x02_P2.54mm_Vertical")
+      (reference "J15") (unit 1) (value "Ports") (footprint "Connector_PinHeader_2.54mm:PinHeader_1x02_P2.54mm_Vertical")
     )
     (path "/d1cc4e83-6665-4554-8c56-a75875a110a4"
-      (reference "J16") (unit 1) (value "Port_access") (footprint "Connector_PinHeader_2.54mm:PinHeader_1x02_P2.54mm_Vertical")
+      (reference "J16") (unit 1) (value "Ports") (footprint "Connector_PinHeader_2.54mm:PinHeader_1x02_P2.54mm_Vertical")
     )
     (path "/e8ad5ff0-8eaa-45eb-ab51-d5714e67e98b"
-      (reference "J17") (unit 1) (value "Port_access") (footprint "Connector_PinHeader_2.54mm:PinHeader_1x02_P2.54mm_Vertical")
+      (reference "J17") (unit 1) (value "Ports") (footprint "Connector_PinHeader_2.54mm:PinHeader_1x02_P2.54mm_Vertical")
     )
     (path "/2ecc3e26-87d0-4ef2-9a29-33be729ac614"
-      (reference "J18") (unit 1) (value "Port_access") (footprint "Connector_PinHeader_2.54mm:PinHeader_1x02_P2.54mm_Vertical")
+      (reference "J18") (unit 1) (value "Ports") (footprint "Connector_PinHeader_2.54mm:PinHeader_1x02_P2.54mm_Vertical")
     )
     (path "/a36b3ac5-f94e-4fd2-9a19-d1032af3fe6c"
-      (reference "J19") (unit 1) (value "Port_access") (footprint "Connector_PinHeader_2.54mm:PinHeader_1x02_P2.54mm_Vertical")
+      (reference "J19") (unit 1) (value "Ports") (footprint "Connector_PinHeader_2.54mm:PinHeader_1x02_P2.54mm_Vertical")
     )
     (path "/37c55c31-4c54-4d44-8006-728f8f061b14"
@@
     )
     (path "/d0f73ae6-0625-401e-8706-a6e20f2f56ef"
-      (reference "J23") (unit 1) (value "Port_access") (footprint "Connector_PinHeader_2.54mm:PinHeader_1x03_P2.54mm_Vertical")
+      (reference "J23") (unit 1) (value "Ports") (footprint "Connector_PinHeader_2.54mm:PinHeader_1x03_P2.54mm_Vertical")
     )
     (path "/97cb558c-de85-4927-b785-7325c3e0be79"
