File: Hardware/PowerSupply_HW/PowerSupply_HW.kicad_pcb (KiCad board)
At the start: 2 copper layers, 102.6 x 97.4 mm, 16 parts, among them J1 PW_Interface, J10 Debug, J11 Debug, J2 AD_Interface, U3 TP4056_MODULE, U4 Modulo_DC-DC_Boost_XL6009

Commit message: geracao de gerbers
Parts:
- removed ? (x2): , 
- removed the REF** at (98.9, 127.2)
- added J3: HighCurrent_Interface, Connector_PinHeader_2.54mm:PinHeader_1x04_P2.54mm_Vertical, F.Cu at (138.0, 68.5)
- added REF**: MountingHole_3mm_Pad, MountingHole:MountingHole_3mm_Pad, F.Cu at (150.7, 40.8)
- added REF**: MountingHole_3mm_Pad, MountingHole:MountingHole_3mm_Pad, F.Cu at (98.9, 124.3)
- added REF**: MountingHole_3mm_Pad, MountingHole:MountingHole_3mm_Pad, F.Cu at (60.1, 66.2)
- renumbered BT1 to Bateria
Routing:
- net +5V: track 58.8 -> 65.6 mm
Other:
- board size 102.6 x 97.4 mm -> 102.6 x 92.9 mm
- board text added: "+-"
