File: Hardware/UserInterface_HW/UserInterface_HW.kicad_pcb (KiCad board)
At the start: 2 copper layers, 108.4 x 84.5 mm, 4 parts, among them J1 Supply, J2 I2C, U1 LCD-PCF8574, U2 LCD-5LC02

Commit message: geracao de gerbers
Parts:
- added ?: , , F.Cu at (92.2, 73.9)
- added ?: , , F.Cu at (180.3, 118.9)
- added ?: , , F.Cu at (90.8, 119.5)
- added REF**: MountingHole_3mm_Pad, MountingHole:MountingHole_3mm_Pad, F.Cu at (180.3, 73.9)
- moved J1 4.11 mm to (91.0, 43.5)
Routing:
- net GNDD: track 34.4 -> 30.3 mm
- net +5V: track 17.7 -> 14.7 mm
- removed copper zone on F.Cu, net GNDD
Other:
- board size 108.4 x 84.5 mm -> 99.4 x 84.6 mm
- board text added: "+-"
- board text added: "DISPLAY 20X4"
- board text added: "SCL SDA"
